File: hardware/TinyMIDI2CV.kicad_sch (KiCad schematic)
At the start: 21 parts, among them J1 HDR-16PIN, J2 MIDI DIN-5, J3 PJ301M-12, J4 PJ301M-12, J5 PJ301M-12, U1 ATtiny85, U2 LM324, U3 6N138

Commit message: Update and rename goMIDI2CV.kicad_sch to TinyMIDI2CV.kicad_sch
Other:
- title: goMIDI2CV -> TinyMIDI2CV
Changed lines of the file:
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@@
   (paper "USLetter")
   (title_block
-    (title "goMIDI2CV")
+    (title "TinyMIDI2CV")
     (date "2023-12-23")
     (rev "3")
@@
     (pin "8")
     (instances
-      (project "goMIDI2CV"
+      (project "TinyMIDI2CV"
         (path "/a2e7f5a5-4bf0-4de9-9dc9-ea0424afec75"
           (reference "U3") (unit 1)
@@
     (pin "5")
     (instances
-      (project "goMIDI2CV"
+      (project "TinyMIDI2CV"
         (path "/a2e7f5a5-4bf0-4de9-9dc9-ea0424afec75"
           (reference "J2") (unit 1)
@@
     (pin "2")
     (instances
-      (project "goMIDI2CV"
+      (project "TinyMIDI2CV"
         (path "/a2e7f5a5-4bf0-4de9-9dc9-ea0424afec75"
           (reference "R3") (unit 1)
@@
     (pin "4")
     (instances
-      (project "goMIDI2CV"
+      (project "TinyMIDI2CV"
         (path "/a2e7f5a5-4bf0-4de9-9dc9-ea0424afec75"
           (reference "U2") (unit 5)
@@
     (pin "3")
     (instances
-      (project "goMIDI2CV"
+      (project "TinyMIDI2CV"
         (path "/a2e7f5a5-4bf0-4de9-9dc9-ea0424afec75"
           (reference "RV1") (unit 1)
@@
     (pin "1")
     (instances
-      (project "goMIDI2CV"
+      (project "TinyMIDI2CV"
         (path "/a2e7f5a5-4bf0-4de9-9dc9-ea0424afec75"
           (reference "#PWR012") (unit 1)
@@
     (pin "TN")
     (instances
-      (project "goMIDI2CV"
+      (project "TinyMIDI2CV"
         (path "/a2e7f5a5-4bf0-4de9-9dc9-ea0424afec75"
           (reference "J3") (unit 1)
@@
     (pin "4")
     (instances
-      (project "goMIDI2CV"
+      (project "TinyMIDI2CV"
         (path "/a2e7f5a5-4bf0-4de9-9dc9-ea0424afec75"
           (reference "U2") (unit 1)
@@
     (pin "1")
     (instances
-      (project "goMIDI2CV"
+      (project "TinyMIDI2CV"
         (path "/a2e7f5a5-4bf0-4de9-9dc9-ea0424afec75"
           (reference "#PWR01") (unit 1)
@@
     (pin "2")
     (instances
-      (project "goMIDI2CV"
+      (project "TinyMIDI2CV"
         (path "/a2e7f5a5-4bf0-4de9-9dc9-ea0424afec75"
           (reference "C4") (unit 1)
@@
     (pin "1")
     (instances
-      (project "goMIDI2CV"
+      (project "TinyMIDI2CV"
         (path "/a2e7f5a5-4bf0-4de9-9dc9-ea0424afec75"
           (reference "#PWR07") (unit 1)
@@
     (pin "1")
     (instances
-      (project "goMIDI2CV"
+      (project "TinyMIDI2CV"
         (path "/a2e7f5a5-4bf0-4de9-9dc9-ea0424afec75"
           (reference "#PWR014") (unit 1)
@@
     (pin "2")
     (instances
-      (project "goMIDI2CV"
+      (project "TinyMIDI2CV"
         (path "/a2e7f5a5-4bf0-4de9-9dc9-ea0424afec75"
           (reference "R7") (unit 1)
@@
     (pin "TN")
     (instances
-      (project "goMIDI2CV"
+      (project "TinyMIDI2CV"
         (path "/a2e7f5a5-4bf0-4de9-9dc9-ea0424afec75"
           (reference "J4") (unit 1)
@@
     (pin "4")
     (instances
-      (project "goMIDI2CV"
+      (project "TinyMIDI2CV"
         (path "/a2e7f5a5-4bf0-4de9-9dc9-ea0424afec75"
           (reference "U2") (unit 4)
@@
     (pin "2")
     (instances
-      (project "goMIDI2CV"
+      (project "TinyMIDI2CV"
         (path "/a2e7f5a5-4bf0-4de9-9dc9-ea0424afec75"
           (reference "R9") (unit 1)
@@
     (pin "2")
     (instances
-      (project "goMIDI2CV"
+      (project "TinyMIDI2CV"
         (path "/a2e7f5a5-4bf0-4de9-9dc9-ea0424afec75"
           (reference "R6") (unit 1)
@@
     (pin "1")
     (instances
-      (project "goMIDI2CV"
+      (project "TinyMIDI2CV"
         (path "/a2e7f5a5-4bf0-4de9-9dc9-ea0424afec75"
           (reference "#PWR013") (unit 1)
@@
     (pin "1")
     (instances
-      (project "goMIDI2CV"
+      (project "TinyMIDI2CV"
         (path "/a2e7f5a5-4bf0-4de9-9dc9-ea0424afec75"
           (reference "#PWR015") (unit 1)
@@
     (pin "8")
     (instances
-      (project "goMIDI2CV"
+      (project "TinyMIDI2CV"
         (path "/a2e7f5a5-4bf0-4de9-9dc9-ea0424afec75"
           (reference "U1") (unit 1)
@@
     (pin "1")
     (instances
-      (project "goMIDI2CV"
+      (project "TinyMIDI2CV"
         (path "/a2e7f5a5-4bf0-4de9-9dc9-ea0424afec75"
           (reference "#PWR08") (unit 1)
@@
     (pin "4")
     (instances
-      (project "goMIDI2CV"
+      (project "TinyMIDI2CV"
         (path "/a2e7f5a5-4bf0-4de9-9dc9-ea0424afec75"
           (reference "U2") (unit 3)
@@
     (pin "9")
     (instances
-      (project "goMIDI2CV"
+      (project "TinyMIDI2CV"
         (path "/a2e7f5a5-4bf0-4de9-9dc9-ea0424afec75"
           (reference "J1") (unit 1)
@@
     (pin "1")
     (instances
-      (project "goMIDI2CV"
+      (project "TinyMIDI2CV"
         (path "/a2e7f5a5-4bf0-4de9-9dc9-ea0424afec75"
           (reference "#PWR011") (unit 1)
@@
     (pin "2")
     (instances
-      (project "goMIDI2CV"
+      (project "TinyMIDI2CV"
         (path "/a2e7f5a5-4bf0-4de9-9dc9-ea0424afec75"
           (reference "R1") (unit 1)
@@
     (pin "2")
     (instances
-      (project "goMIDI2CV"
+      (project "TinyMIDI2CV"
         (path "/a2e7f5a5-4bf0-4de9-9dc9-ea0424afec75"
           (reference "D1") (unit 1)
@@
     (pin "1")
     (instances
-      (project "goMIDI2CV"
+      (project "TinyMIDI2CV"
         (path "/a2e7f5a5-4bf0-4de9-9dc9-ea0424afec75"
           (reference "#PWR09") (unit 1)
@@
     (pin "4")
     (instances
-      (project "goMIDI2CV"
+      (project "TinyMIDI2CV"
         (path "/a2e7f5a5-4bf0-4de9-9dc9-ea0424afec75"
           (reference "U2") (unit 2)
@@
     (pin "1")
     (instances
-      (project "goMIDI2CV"
+      (project "TinyMIDI2CV"
         (path "/a2e7f5a5-4bf0-4de9-9dc9-ea0424afec75"
           (reference "#PWR04") (unit 1)
@@
     (pin "1")
     (instances
-      (project "goMIDI2CV"
+      (project "TinyMIDI2CV"
         (path "/a2e7f5a5-4bf0-4de9-9dc9-ea0424afec75"
           (reference "#PWR05") (unit 1)
@@
     (pin "1")
     (instances
-      (project "goMIDI2CV"
+      (project "TinyMIDI2CV"
         (path "/a2e7f5a5-4bf0-4de9-9dc9-ea0424afec75"
           (reference "#PWR02") (unit 1)
@@
     (pin "1")
     (instances
-      (project "goMIDI2CV"
+      (project "TinyMIDI2CV"
         (path "/a2e7f5a5-4bf0-4de9-9dc9-ea0424afec75"
           (reference "#PWR06") (unit 1)
@@
     (pin "TN")
     (instances
-      (project "goMIDI2CV"
+      (project "TinyMIDI2CV"
         (path "/a2e7f5a5-4bf0-4de9-9dc9-ea0424afec75"
           (reference "J5") (unit 1)
@@
     (pin "2")
     (instances
-      (project "goMIDI2CV"
+      (project "TinyMIDI2CV"
         (path "/a2e7f5a5-4bf0-4de9-9dc9-ea0424afec75"
           (reference "R8") (unit 1)
@@
     (pin "2")
     (instances
-      (project "goMIDI2CV"
+      (project "TinyMIDI2CV"
         (path "/a2e7f5a5-4bf0-4de9-9dc9-ea0424afec75"
           (reference "R4") (unit 1)
@@
     (pin "1")
     (instances
-      (project "goMIDI2CV"
+      (project "TinyMIDI2CV"
         (path "/a2e7f5a5-4bf0-4de9-9dc9-ea0424afec75"
           (reference "#PWR03") (unit 1)
@@
     (pin "2")
     (instances
-      (project "goMIDI2CV"
+      (project "TinyMIDI2CV"
         (path "/a2e7f5a5-4bf0-4de9-9dc9-ea0424afec75"
           (reference "R5") (unit 1)
@@
     (pin "1")
     (instances
-      (project "goMIDI2CV"
+      (project "TinyMIDI2CV"
         (path "/a2e7f5a5-4bf0-4de9-9dc9-ea0424afec75"
           (reference "#PWR016") (unit 1)
@@
     (pin "2")
     (instances
-      (project "goMIDI2CV"
+      (project "TinyMIDI2CV"
         (path "/a2e7f5a5-4bf0-4de9-9dc9-ea0424afec75"
           (reference "C2") (unit 1)
@@
     (pin "2")
     (instances
-      (project "goMIDI2CV"
+      (project "TinyMIDI2CV"
         (path "/a2e7f5a5-4bf0-4de9-9dc9-ea0424afec75"
           (reference "R2") (unit 1)
@@
     (pin "1")
     (instances
-      (project "goMIDI2CV"
+      (project "TinyMIDI2CV"
         (path "/a2e7f5a5-4bf0-4de9-9dc9-ea0424afec75"
           (reference "#PWR010") (unit 1)
